Commit message: igibson --> omnigibson

File: igibson/examples/ros/igibson-ros/turtlebot/turtlebot.urdf (robot description, URDF)
Before this commit: robot turtlebot, 36 links, 35 joints
Links:
- link base_link: geometry collision cylinder length=0.10938 radius=0.176; visual mesh filename=package://omnigibson-ros/turtlebot/kobuki_description/meshe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
- link kinect_camera: geometry collision box size=0.07271 0.27794 0.073; visual mesh filename=package://omnigibson-ros/turtlebot/turtlebot_description/me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
- link plate_bottom_link: geometry collision box size=0.26727 0.340 0.006; visual mesh filename=package://omnigibson-ros/turtlebot/turtlebot_description/me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
- link plate_middle_link: geometry collision box size=0.28727 0.340 0.006; visual mesh filename=package://omnigibson-ros/turtlebot/turtlebot_description/me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
- link plate_top_link: geometry collision box size=0.28727 0.340 0.006; visual mesh filename=package://omnigibson-ros/turtlebot/turtlebot_description/me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
- link pole_bottom_0_link: geometry collision cylinder length=0.0492 radius=.006; visual mesh filename=package://omnigibson-ros/turtlebot/turtlebot_description/me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
- link pole_bottom_1_link: geometry collision cylinder length=0.0492 radius=.006; visual mesh filename=package://omnigibson-ros/turtlebot/turtlebot_description/me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
- link pole_bottom_2_link: geometry collision cylinder length=0.0492 radius=.006; visual mesh filename=package://omnigibson-ros/turtlebot/turtlebot_description/me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
- link pole_bottom_3_link: geometry collision cylinder length=0.0492 radius=.006; visual mesh filename=package://omnigibson-ros/turtlebot/turtlebot_description/me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
- link pole_bottom_4_link: geometry collision cylinder length=0.0492 radius=.006; visual mesh filename=package://omnigibson-ros/turtlebot/turtlebot_description/me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
- link pole_bottom_5_link: geometry collision cylinder length=0.0492 radius=.006; visual mesh filename=package://omnigibson-ros/turtlebot/turtlebot_description/me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
- link pole_kinect_0_link: geometry collision cylinder length=0.0936 radius=0.006; visual mesh filename=package://omnigibson-ros/turtlebot/turtlebot_description/me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
- link pole_kinect_1_link: geometry collision cylinder length=0.0936 radius=0.006; visual mesh filename=package://omnigibson-ros/turtlebot/turtlebot_description/me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
- link pole_middle_0_link: geometry collision cylinder length=0.0608 radius=.006; visual mesh filename=package://omnigibson-ros/turtlebot/turtlebot_description/me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
- link pole_middle_1_link: geometry collision cylinder length=0.0608 radius=.006; visual mesh filename=package://omnigibson-ros/turtlebot/turtlebot_description/me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
- link pole_middle_2_link: geometry collision cylinder length=0.0608 radius=.006; visual mesh filename=package://omnigibson-ros/turtlebot/turtlebot_description/me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
- link pole_middle_3_link: geometry collision cylinder length=0.0608 radius=.006; visual mesh filename=package://omnigibson-ros/turtlebot/turtlebot_description/me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
- link pole_top_0_link: geometry collision cylinder length=0.2032 radius=.006; visual mesh filename=package://omnigibson-ros/turtlebot/turtlebot_description/me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
- link pole_top_1_link: geometry collision cylinder length=0.2032 radius=.006; visual mesh filename=package://omnigibson-ros/turtlebot/turtlebot_description/me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
- link pole_top_2_link: geometry collision cylinder length=0.2032 radius=.006; visual mesh filename=package://omnigibson-ros/turtlebot/turtlebot_description/me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
- link pole_top_3_link: geometry collision cylinder length=0.2032 radius=.006; visual mesh filename=package://omnigibson-ros/turtlebot/turtlebot_description/me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
- link wheel_left_link: geometry collision cylinder length=0.0206 radius=0.0352; visual mesh filename=package://omnigibson-ros/turtlebot/kobuki_description/meshe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
- link wheel_right_link: geometry collision cylinder length=0.0206 radius=0.0350; visual mesh filename=package://omnigibson-ros/turtlebot/kobuki_description/meshe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
